File: pcbs/AudioPlayground_HeadsetShield/AudioPlayground_HeadsetShield.kicad_pcb (KiCad board)
At the start: 2 copper layers, 20.1 x 22.9 mm, 9 parts, among them J1 Conn_01x05_Socket, J3 SJ2-35364B-SMT-TR, J4 SJ2-35364B-SMT-TR, J9 Conn_01x05_Socket, SW1 SW_Push, SW2 SW_Push, SW3 SW_Push, SW4 SW_Push, SW5 SW_Push

Commit message: Add HeadsetShield v2.0
Parts:
- removed J1, J9: Conn_01x05_Socket, Connector_PinHeader_2.54mm:PinHeader_1x07_P2.54mm_Vertical
- removed J3, J4: SJ2-35364B-SMT-TR, SJ235364BSMTTR:SJ235364BSMTTR
- added CN1: PJ-342, PJ-342:PJ-342, F.Cu at (128.4, 99.7)
- added CN2: PJ-342, PJ-342:PJ-342, F.Cu at (128.4, 111.4)
- added G***: LOGO, LOGO, B.Cu at (126.1, 106.4)
- added J2: Conn_01x07_Socket, Connector_PinHeader_2.54mm:PinHeader_1x07_P2.54mm_Vertical_SMD_Pin1Left, B.Cu at (124.1, 95.4)
- added J5: Conn_01x07_Socket, Connector_PinHeader_2.54mm:PinHeader_1x07_P2.54mm_Vertical_SMD_Pin1Left, B.Cu at (124.1, 115.7)
- added JP1: Jumper_2_Bridged, Jumper:SolderJumper-2_P1.3mm_Bridged2Bar_RoundedPad1.0x1.5mm, B.Cu at (129.2, 111.0)
- added SW6: 7*7*5-6P-L WX, 7*7*5-6P-LWX:7*7*5-6P-LWX, F.Cu at (118.8, 105.6)
- moved SW4 7.40 mm to (117.1, 94.6), turned to 90 degrees
- moved SW3 6.91 mm to (120.7, 99.1), turned to 0 degrees
- moved SW1 5.22 mm to (120.4, 117.2)
- moved SW5 5.17 mm to (121.4, 94.6), turned to 90 degrees
- moved SW2 4.57 mm to (120.4, 112.9)
Routing:
- net /BTN1: track 22.1 -> 45.0 mm
- net /ROUTP: track 2.34 -> 22.9 mm, vias 0 -> 1
- net /BTN5: track 3.88 -> 18.7 mm, vias 0 -> 2
- net /BTN4: track 8.82 -> 23.2 mm, vias 0 -> 1
- net /LINL: track 19.5 -> 9.48 mm
- net /MIC: track 12.0 -> 21.7 mm, vias 1 -> 2
- net /BTN3: track 13.0 -> 21.3 mm, vias 0 -> 1
- net /JACKSNS: track 10.00 -> 3.83 mm, vias 1 -> 0
- net /BTN2: track 17.7 -> 21.5 mm, vias 0 -> 1
- net /LINR: track 14.1 -> 11.9 mm
- net /LOUTP: track 10.9 -> 12.2 mm, vias 0 -> 1
- net GND: vias 20 -> 6
Other:
- board size 20.1 x 22.9 mm -> 20.1 x 27.2 mm
- board text added: "4"
- board text added: "5"
- board text added: "HEADSET"
- board text added: "HeadsetShield v2.0"
- board text added: "LINE IN"
- board text removed: "BTN4"
- board text removed: "BTN5"

Commit message: Fix Naming
Parts:
- SW6: value 7*7*5-6P-L WX -> 775-6P-LWX
Changed lines of the file:
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@@
 			)
 		)
-		(property "Value" "7*7*5-6P-L WX"
+		(property "Value" "775-6P-LWX"
 			(at 0 8 135)
 			(layer "F.Fab")
@@
 		)
 		(embedded_fonts no)
-		(model "${KIPRJMOD}/../../components/7*7*5-6P-LWX/7*7*5-6P-LWX.step"
+		(model "${KIPRJMOD}/../../components/775-6P-LWX/775-6P-LWX.step"
 			(offset
 				(xyz 0 -0 1.8)
@@
 		(sheetfile "AudioPlayground_HeadsetShield.kicad_sch")
 		(zone_connect 1)
-		(attr exclude_from_pos_files exclude_from_bom allow_soldermask_bridges)
+		(attr exclude_from_pos_files allow_soldermask_bridges)
 		(net_tie_pad_groups "1, 2")
 		(fp_poly

Commit message: Fix Headset Shield
Parts:
- SW6: footprint 7*7*5-6P-LWX:7*7*5-6P-LWX -> 775-6P-LWX:775-6P-LWX
Connections:
- CN1 pad 2: GND -> /MIC
- CN1 pad 3: /MIC -> GND
- SW6 pad 1: /BTN1 -> /BTN2
- SW6 pad 4: /BTN2 -> /BTN1
Routing:
- net /BTN1: track 45.0 -> 37.4 mm
- net /MIC: track 21.7 -> 29.0 mm
- net /BTN2: track 21.5 -> 27.1 mm, vias 1 -> 2
Changed lines of the file:
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@@
 	(net 17 "unconnected-(CN2-Pad7)")
 	(net 18 "unconnected-(CN2-Pad6)")
-	(footprint "7*7*5-6P-LWX:7*7*5-6P-LWX"
+	(footprint "775-6P-LWX:775-6P-LWX"
 		(layer "F.Cu")
 		(at 118.776 105.581262 -45)
 		(property "Reference" "SW6"
-			(at 0 -8 135)
+			(at 0 -8 315)
 			(layer "F.SilkS")
-			(hide yes)
 			(effects
 				(font
@@
 		)
 		(property "Value" "775-6P-LWX"
-			(at 0 8 135)
+			(at 0 8 315)
 			(layer "F.Fab")
-			(hide yes)
 			(effects
 				(font
@@
 		)
 		(property "Datasheet" ""
-			(at 0 0 135)
+			(at 0 0 315)
 			(layer "F.Fab")
 			(hide yes)
@@
 		)
 		(property "Description" ""
-			(at 0 0 135)
+			(at 0 0 315)
 			(layer "F.Fab")
 			(hide yes)
@@
 		(attr smd)
 		(fp_line
+			(start -3.5 3.5)
+			(end -3.5 2.13)
+			(stroke
+				(width 0.25)
+				(type solid)
+			)
+			(layer "F.SilkS")
+		)
+		(fp_line
+			(start -3.5 3.5)
+			(end -0.98 3.5)
+			(stroke
+				(width 0.25)
+				(type solid)
+			)
+			(layer "F.SilkS")
+		)
+		(fp_line
+			(start -0.84 3.29)
+			(end 0 2.450001)
+			(stroke
+				(width 0.25)
+				(type solid)
+			)
+			(layer "F.SilkS")
+		)
+		(fp_line
+			(start 0.98 3.5)
+			(end 3.5 3.5)
+			(stroke
+				(width 0.25)
+				(type solid)
+			)
+			(layer "F.SilkS")
+		)
+		(fp_line
+			(start 0 2.450001)
+			(end 0.84 3.29)
+			(stroke
+				(width 0.25)
+				(type solid)
+			)
+			(layer "F.SilkS")
+		)
+		(fp_line
+			(start -3.5 -2.13)
+			(end -3.5 -3.5)
+			(stroke
+				(width 0.25)
+				(type solid)
+			)
+			(layer "F.SilkS")
+		)
+		(fp_line
 			(start -0.7 0)
 			(end -0.7 0)
@@
 			(layer "F.SilkS")
 		)
+		(fp_line
+			(start 3.5 2.13)
+			(end 3.5 3.5)
+			(stroke
+				(width 0.25)
+				(type solid)
+			)
+			(layer "F.SilkS")
+		)
+		(fp_line
+			(start -0.98 -3.5)
+			(end -3.5 -3.5)
+			(stroke
+				(width 0.25)
+				(type solid)
+			)
+			(layer "F.SilkS")
+		)
+		(fp_line
+			(start 3.5 -3.5)
+			(end 0.98 -3.5)
+			(stroke
+				(width 0.25)
+				(type solid)
+			)
+			(layer "F.SilkS")
+		)
+		(fp_line
+			(start 3.5 -3.5)
+			(end 3.5 -2.13)
+			(stroke
+				(width 0.25)
+				(type solid)
+			)
+			(layer "F.SilkS")
+		)
 		(fp_arc
 			(start -0.63 1.36)
@@
 		)
 		(fp_text user "${REFERENCE}"
-			(at 0 0 135)
+			(at 0 0 315)
 			(layer "F.Fab")
 			(effects
@@
 			(size 1.5 1)
 			(layers "F.Cu" "F.Mask" "F.Paste")
-			(net 11 "/BTN1")
+			(net 13 "/BTN2")
 			(pinfunction "1")
 			(pintype "unspecified")
@@
 			(size 1.5 1)
 			(layers "F.Cu" "F.Mask" "F.Paste")
-			(net 13 "/BTN2")
+			(net 11 "/BTN1")
 			(pinfunction "4")
 			(pintype "unspecified")
@@
 		)
 		(embedded_fonts no)
-		(model "${KIPRJMOD}/../../components/775-6P-LWX/775-6P-LWX.step"
+		(model "${EASYEDA2KICAD}/easyeda2kicad.3dshapes/SW-SMD_8P-L7.0-W7.0-P1.40-LS7.4-TL.wrl"
 			(offset
-				(xyz 0 -0 1.8)
+				(xyz 0 -0 0.6)
 			)
 			(scale
@@
 			)
 			(rotate
-				(xyz -0 -0 180)
+				(xyz 0 0 180)
 			)
 		)
@@
 			(size 2.3 1.6)
 			(layers "F.Cu" "F.Mask" "F.Paste")
-			(net 1 "GND")
+			(net 4 "/MIC")
 			(pinfunction "2")
 			(pintype "unspecified")
@@
 			(size 2.3 1.6)
 			(layers "F.Cu" "F.Mask" "F.Paste")
-			(net 4 "/MIC")
+			(net 1 "GND")
 			(pinfunction "3")
 			(pintype "unspecified")
@@
 	)
 	(segment
-		(start 130.8918 109.457)
-		(end 128.7328 109.457)
+		(start 131.5014 108.8474)
+		(end 131.5014 97.4428)
 		(width 0.2)
 		(layer "F.Cu")
@@
 	)
 	(segment
-		(start 133.0238 103.3204)
-		(end 131.5014 104.8428)
+		(start 128.7328 109.457)
+		(end 130.8918 109.457)
 		(width 0.2)
 		(layer "F.Cu")
@@
 	)
 	(segment
-		(start 131.5014 104.8428)
+		(start 130.8918 109.457)
 		(end 131.5014 108.8474)
 		(width 0.2)
@@
 	)
 	(segment
-		(start 131.5014 108.8474)
-		(end 130.8918 109.457)
+		(start 131.5014 97.4428)
+		(end 132.9238 96.0204)
 		(width 0.2)
 		(layer "F.Cu")
@@
 	)
 	(segment
-		(start 122.0508 117.1532)
-		(end 122.0508 115.8088)
+		(start 122.0526 115.807)
+		(end 121.09 114.8444)
 		(width 0.2)
 		(layer "F.Cu")
@@
 	)
 	(segment
-		(start 122.0508 115.8088)
-		(end 122.0526 115.807)
+		(start 122.0508 117.1532)
+		(end 122.0508 115.8088)
 		(width 0.2)
 		(layer "F.Cu")
@@
 	)
 	(segment
-		(start 118.4204 103.245763)
-		(end 118.4204 110.979)
+		(start 121.09 109.875161)
+		(end 120.084148 108.869309)
 		(width 0.2)
 		(layer "F.Cu")
@@
 	)
 	(segment
-		(start 122.0526 114.6112)
+		(start 122.0508 115.8088)
 		(end 122.0526 115.807)
 		(width 0.2)
@@
 	)
 	(segment
-		(start 118.4204 110.979)
-		(end 122.0526 114.6112)
-		(width 0.2)
-		(layer "F.Cu")
-		(net 11)
-	)
-	(segment
-		(start 117.467852 102.293215)
-		(end 118.4204 103.245763)
+		(start 121.09 114.8444)
+		(end 121.09 109.875161)
 		(width 0.2)
 		(layer "F.Cu")
@@
 	)
 	(segment
-		(start 121.738639 110.5238)
-		(end 122.078 110.5238)
+		(start 118.4046 103.48)
+		(end 118.4046 103.229963)
 		(width 0.2)
 		(layer "F.Cu")
@@
 	)
 	(segment
-		(start 122.078 110.5238)
-		(end 122.0508 110.551)
+		(start 118.4046 103.229963)
+		(end 117.467852 102.293215)
 		(width 0.2)
 		(layer "F.Cu")
@@
 	)
 	(segment
-		(start 122.0508 110.551)
-		(end 122.0508 112.9114)
+		(start 122.078 110.5238)
+		(end 122.0508 110.551)
 		(width 0.2)
 		(layer "F.Cu")
@@
 	)
 	(segment
-		(start 120.084148 108.869309)
-		(end 121.738639 110.5238)
+		(start 122.0508 110.551)
+		(end 122.0508 112.9114)
 		(width 0.2)
 		(layer "F.Cu")
@@
 		(net 13)
 	)
+	(via
+		(at 118.4046 103.48)
+		(size 0.6)
+		(drill 0.3)
+		(layers "F.Cu" "B.Cu")
+		(net 13)
+	)
+	(segment
+		(start 122.078 108.468)
+		(end 122.078 108.68)
+		(width 0.2)
+		(layer "B.Cu")
+		(net 13)
+	)
 	(segment
 		(start 126.4468 100.9734)
@@
 	(segment
 		(start 122.078 105.3422)
+		(end 122.078 108.68)
+		(width 0.2)
+		(layer "B.Cu")
+		(net 13)
+	)
+	(segment
+		(start 122.078 108.68)
 		(end 122.078 110.5238)
 		(width 0.2)
@@
 	)
 	(segment
+		(start 118.4046 104.7946)
+		(end 122.078 108.468)
+		(width 0.2)
+		(layer "B.Cu")
+		(net 13)
+	)
+	(segment
 		(start 129.19 97.0444)
 		(end 129.19 98.2302)
 		(width 0.2)
 		(layer "B.Cu")
+		(net 13)
+	)
+	(segment
+		(start 118.4046 103.48)
+		(end 118.4046 104.7946)
+		(width 0.2)
+		(layer "B.Cu")

Commit message: Fix Joystick
Connections:
- SW6 pad 3: /BTN5 -> /BTN4
- SW6 pad 6: /BTN4 -> /BTN5
Routing:
- net /BTN4: track 23.2 -> 17.4 mm
- net /BTN5: track 18.7 -> 20.4 mm
Changed lines of the file:
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@@
 			(size 1.5 1)
 			(layers "F.Cu" "F.Mask" "F.Paste")
-			(net 10 "/BTN5")
+			(net 12 "/BTN4")
 			(pinfunction "3")
 			(pintype "unspecified")
@@
 			(size 1.5 1)
 			(layers "F.Cu" "F.Mask" "F.Paste")
-			(net 12 "/BTN4")
+			(net 10 "/BTN5")
 			(pinfunction "6")
 			(pintype "unspecified")
@@
 	)
 	(segment
-		(start 121.5954 96.1456)
-		(end 121.443 96.298)
+		(start 120.2746 102.8784)
+		(end 120.2746 102.8646)
 		(width 0.2)
 		(layer "F.Cu")
@@
 	)
 	(segment
-		(start 115.497114 104.273114)
-		(end 116.4646 105.2406)
+		(start 121.5954 96.1456)
+		(end 121.443 96.298)
 		(width 0.2)
 		(layer "F.Cu")
@@
 	)
 	(segment
-		(start 115.487953 104.273114)
-		(end 115.497114 104.273114)
+		(start 122.064047 106.88941)
+		(end 122.064047 104.667847)
 		(width 0.2)
 		(layer "F.Cu")
@@
 		(net 10)
 	)
+	(segment
+		(start 120.2746 102.8646)
+		(end 119.99 102.58)
+		(width 0.2)
+		(layer "F.Cu")
+		(net 10)
+	)
+	(segment
+		(start 122.064047 104.667847)
+		(end 120.2746 102.8784)
+		(width 0.2)
+		(layer "F.Cu")
+		(net 10)
+	)
 	(via
-		(at 116.4646 105.2406)
+		(at 121.5954 95.5124)
 		(size 0.45)
 		(drill 0.3)
@@
 	)
 	(via
-		(at 121.5954 95.5124)
-		(size 0.45)
+		(at 119.99 102.58)
+		(size 0.6)
 		(drill 0.3)
 		(layers "F.Cu" "B.Cu")
@@
 	)
 	(segment
+		(start 117.563762 95.853762)
+		(end 119.683123 93.7344)
+		(width 0.2)
+		(layer "B.Cu")
+		(net 10)
+	)
+	(segment
 		(start 121.57 93.7344)
 		(end 121.57 95.487)
@@
 	)
 	(segment
-		(start 116.4646 96.952923)
-		(end 119.683123 93.7344)
+		(start 119.99 102.58)
+		(end 117.563762 100.153762)
 		(width 0.2)
 		(layer "B.Cu")
@@
 	)
 	(segment
-		(start 116.4646 105.2406)
-		(end 116.4646 96.952923)
+		(start 117.563762 100.153762)
+		(end 117.563762 95.853762)
 		(width 0.2)
 		(layer "B.Cu")
@@
 	)
 	(segment
-		(start 122.064047 106.88941)
-		(end 122.064047 104.667847)
-		(width 0.2)
-		(layer "F.Cu")
-		(net 12)
-	)
-	(segment
-		(start 119.1552 96.3488)
-		(end 117.125 96.3488)
+		(start 114.89 103.675161)
+		(end 115.186953 103.972114)
 		(width 0.2)
 		(layer "F.Cu")
@@
 	)
 	(segment
-		(start 120.2746 102.0402)
-		(end 121.443 100.8718)
+		(start 114.89 102.18)
+		(end 114.89 103.675161)
 		(width 0.2)
 		(layer "F.Cu")
@@
 	)
 	(segment
-		(start 121.443 98.6366)
-		(end 119.1552 96.3488)
+		(start 115.487953 104.273114)
+		(end 115.497114 104.273114)
 		(width 0.2)
 		(layer "F.Cu")
@@
 	)
 	(segment
-		(start 120.2746 102.8784)
-		(end 120.2746 102.0402)
+		(start 117.8634 96.298)
+		(end 117.125 96.298)
 		(width 0.2)
 		(layer "F.Cu")
@@
 	)
 	(segment
-		(start 117.8634 96.298)
-		(end 117.125 96.298)
+		(start 119.2586 94.9028)
+		(end 117.8634 96.298)
 		(width 0.2)
 		(layer "F.Cu")
@@
 	)
 	(segment
-		(start 119.2586 94.9028)
-		(end 117.8634 96.298)
+		(start 117.125 99.945)
+		(end 114.89 102.18)
 		(width 0.2)
 		(layer "F.Cu")
@@
 	)
 	(segment
-		(start 121.443 100.8718)
-		(end 121.443 98.6366)
+		(start 117.125 96.3488)
+		(end 117.125 99.945)
 		(width 0.2)
 		(layer "F.Cu")
@@
 	)
 	(segment
-		(start 122.064047 104.667847)
-		(end 120.2746 102.8784)
+		(start 115.186953 103.972114)
+		(end 115.487953 103.972114)
 		(width 0.2)
 		(layer "F.Cu")

Commit message: Add Gerbers
Other:
- board text added: "HeadsetShield v2.1"
- board text removed: "HeadsetShield v2.0"
Changed lines of the file:
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@@
 		)
 	)
-	(gr_text "HeadsetShield\nv2.0"
+	(gr_text "HeadsetShield\nv2.1"
 		(at 133.3556 104.3516 0)
 		(layer "B.SilkS")
