File: pcbs/AudioPlayground_HeadsetShield/AudioPlayground_HeadsetShield.kicad_sch (KiCad schematic)
At the start: 9 parts, among them J1 Conn_01x05_Socket, J3 SJ2-35364B-SMT-TR, J4 SJ2-35364B-SMT-TR, J9 Conn_01x05_Socket, SW1 SW_Push, SW2 SW_Push, SW3 SW_Push, SW4 SW_Push, SW5 SW_Push

Commit message: Add HeadsetShield v2.0
Parts:
- removed J1, J9: Conn_01x05_Socket, Connector_PinHeader_2.54mm:PinHeader_1x07_P2.54mm_Vertical, symbol Connector:Conn_01x07_Pin
- removed J3, J4: SJ2-35364B-SMT-TR, SJ235364BSMTTR:SJ235364BSMTTR, symbol Connector_Audio:AudioJack4_SwitchT1
- added CN1, CN2: PJ-342, PJ-342:PJ-342, symbol PJ-342:PJ-342
- added J2, J5: Conn_01x07_Socket, Connector_PinHeader_2.54mm:PinHeader_1x07_P2.54mm_Vertical_SMD_Pin1Left, symbol Connector:Conn_01x07_Pin
- added JP1: Jumper_2_Bridged, Jumper:SolderJumper-2_P1.3mm_Bridged2Bar_RoundedPad1.0x1.5mm, symbol Jumper:Jumper_2_Bridged
- added SW6: 7*7*5-6P-L WX, 7*7*5-6P-LWX:7*7*5-6P-LWX, symbol 7*7*5-6P-LWX:7*7*5-6P-LWX
- SW1, SW2, SW3, SW4, SW5: LCSC (none) -> C231329
Connections:
- net +3.3V: now also J2.2 (Pin_2)
- net BTN1: now also J2.7 (Pin_7), SW6.1
- net BTN2: now also J2.6 (Pin_6), SW6.4
- net BTN3: now also J2.5 (Pin_5), SW6.5
- net BTN4: now also J2.4 (Pin_4), SW6.6
- net BTN5: now also J2.3 (Pin_3), SW6.3
- net GND: now also CN1.2, CN2.2, CN2.3, J5.1 (Pin_1), SW6.2
- net JACKSNS: now also J5.7 (Pin_7), JP1.2 (B)
- net LINL: now also CN2.5, J5.2 (Pin_2)
- net LINR: now also CN2.4, J5.3 (Pin_3)
- net LOUTP: now also CN1.5, J5.5 (Pin_5)
- net MIC: now also CN1.3, J5.4 (Pin_4), JP1.1 (A)
- net ROUTP: now also CN1.4, J5.6 (Pin_6)
- net VHI: now also J2.1 (Pin_1)
- no-connect marks 1 -> 4
Other:
- note added: "(CTIA STD)"
- moved on the sheet: SW1, SW2, SW3, SW4, SW5

Commit message: Fix Naming
Parts:
- SW6: value 7*7*5-6P-L WX -> 775-6P-LWX; footprint 7*7*5-6P-LWX:7*7*5-6P-LWX -> 775-6P-LWX:775-6P-LWX
Changed lines of the file:
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@@
 			)
 		)
-		(property "Value" "7*7*5-6P-L WX"
+		(property "Value" "775-6P-LWX"
 			(at 154.94 120.65 0)
 			(effects
@@
 			)
 		)
-		(property "Footprint" "7*7*5-6P-LWX:7*7*5-6P-LWX"
+		(property "Footprint" "775-6P-LWX:775-6P-LWX"
 			(at 154.94 143.51 0)
 			(effects

Commit message: Fix Headset Shield
Connections:
- net BTN1: now also SW6.4; no longer SW6.1
- net BTN2: now also SW6.1; no longer SW6.4
- net GND: now also CN1.3; no longer CN1.2
- net MIC: now also CN1.2; no longer CN1.3
Other:
- moved on the sheet: JP1
Changed lines of the file:
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@@
 	(text "(CTIA STD)"
 		(exclude_from_sim no)
-		(at 130.81 99.568 0)
+		(at 130.81 86.868 0)
 		(effects
 			(font
@@
 		)
 	)
+	(wire
+		(pts
+			(xy 113.03 107.95) (xy 113.03 109.22)
+		)
+		(stroke
+			(width 0)
+			(type default)
+		)
+	)
 	(bus
 		(pts
@@
 	(wire
 		(pts
+			(xy 111.76 95.25) (xy 125.73 95.25)
+		)
+		(stroke
+			(width 0)
+			(type default)
+		)
+	)
+	(wire
+		(pts
 			(xy 130.81 130.81) (xy 142.24 130.81)
 		)
@@
 	(wire
 		(pts
-			(xy 113.03 93.98) (xy 113.03 95.25)
-		)
-		(stroke
-			(width 0)
-			(type default)
-		)
-	)
-	(wire
-		(pts
 			(xy 120.65 62.23) (xy 104.14 62.23)
 		)
@@
 	(wire
 		(pts
-			(xy 113.03 95.25) (xy 111.76 95.25)
-		)
-		(stroke
-			(width 0)
-			(type default)
-		)
-	)
-	(wire
-		(pts
 			(xy 172.72 125.73) (xy 167.64 125.73)
 		)
@@
 	(wire
 		(pts
+			(xy 149.86 95.25) (xy 135.89 95.25)
+		)
+		(stroke
+			(width 0)
+			(type default)
+		)
+	)
+	(wire
+		(pts
 			(xy 195.58 93.98) (xy 195.58 102.87)
 		)
@@
 	(wire
 		(pts
-			(xy 149.86 107.95) (xy 135.89 107.95)
-		)
-		(stroke
-			(width 0)
-			(type default)
-		)
-	)
-	(wire
-		(pts
 			(xy 195.58 102.87) (xy 195.58 105.41)
 		)
@@
 	(wire
 		(pts
-			(xy 111.76 107.95) (xy 125.73 107.95)
-		)
-		(stroke
-			(width 0)
-			(type default)
-		)
-	)
-	(wire
-		(pts
 			(xy 137.16 125.73) (xy 142.24 125.73)
 		)
@@
 		(pts
 			(xy 104.14 64.77) (xy 113.03 64.77)
+		)
+		(stroke
+			(width 0)
+			(type default)
+		)
+	)
+	(wire
+		(pts
+			(xy 111.76 107.95) (xy 113.03 107.95)
 		)
 		(stroke
@@
 		)
 	)
-	(label "BTN1"
-		(at 137.16 125.73 0)
-		(effects
-			(font
-				(size 1.27 1.27)
-			)
-			(justify left bottom)
-		)
-	)
 	(label "BTN3"
 		(at 184.15 85.09 0)
@@
 		)
 	)
-	(label "JACKSNS"
-		(at 149.86 107.95 180)
-		(effects
-			(font
-				(size 1.27 1.27)
-			)
-			(justify right bottom)
-		)
-	)
 	(label "MIC"
 		(at 140.97 67.31 180)
@@
 		)
 	)
+	(label "JACKSNS"
+		(at 149.86 95.25 180)
+		(effects
+			(font
+				(size 1.27 1.27)
+			)
+			(justify right bottom)
+		)
+	)
 	(label "BTN2"
 		(at 184.15 93.98 0)
@@
 	)
 	(label "MIC"
-		(at 116.84 107.95 180)
+		(at 119.38 95.25 180)
 		(effects
 			(font
@@
 		)
 	)
-	(label "BTN2"
-		(at 172.72 135.89 180)
-		(effects
-			(font
-				(size 1.27 1.27)
-			)
-			(justify right bottom)
-		)
-	)
 	(label "ROUTP"
 		(at 140.97 72.39 180)
@@
 		)
 	)
+	(label "BTN2"
+		(at 137.16 125.73 0)
+		(effects
+			(font
+				(size 1.27 1.27)
+			)
+			(justify left bottom)
+		)
+	)
 	(label "{BTN[1..5]}"
 		(at 116.84 77.47 0)
@@
 	(label "BTN3"
 		(at 113.03 69.85 180)
+		(effects
+			(font
+				(size 1.27 1.27)
+			)
+			(justify right bottom)
+		)
+	)
+	(label "BTN1"
+		(at 172.72 135.89 180)
 		(effects
 			(font
@@
 	(symbol
 		(lib_id "power:GND")
-		(at 113.03 93.98 180)
+		(at 113.03 109.22 0)
 		(unit 1)
 		(exclude_from_sim no)
@@
 		(on_board yes)
 		(dnp no)
-		(fields_autoplaced yes)
 		(property "Reference" "#PWR02"
-			(at 113.03 87.63 0)
+			(at 113.03 115.57 0)
 			(effects
 				(font
@@
 		)
 		(property "Value" "GND"
-			(at 113.03 88.9 0)
-			(effects
-				(font
-					(size 1.27 1.27)
-				)
+			(at 115.062 110.49 0)
+			(effects
+				(font
+					(size 1.27 1.27)
+				)
+				(justify left)
 			)
 		)
 		(property "Footprint" ""
-			(at 113.03 93.98 0)
+			(at 113.03 109.22 0)
 			(effects
 				(font
@@
 		)
 		(property "Datasheet" ""
-			(at 113.03 93.98 0)
+			(at 113.03 109.22 0)
 			(effects
 				(font
@@
 		)
 		(property "Description" "Power symbol creates a global label with name \"GND\" , ground"
-			(at 113.03 93.98 0)
+			(at 113.03 109.22 0)
 			(effects
 				(font
@@
 	(symbol
 		(lib_id "Jumper:Jumper_2_Bridged")
-		(at 130.81 107.95 0)
+		(at 130.81 95.25 0)
 		(unit 1)
 		(exclude_from_sim no)
@@
 		(fields_autoplaced yes)
 		(property "Reference" "JP1"
-			(at 130.81 102.87 0)
+			(at 130.81 90.17 0)
 			(effects
 				(font
@@
 		)
 		(property "Value" "Jumper_2_Bridged"
-			(at 130.81 105.41 0)
+			(at 130.81 92.71 0)
 			(effects
 				(font
@@
 		)
 		(property "Footprint" "Jumper:SolderJumper-2_P1.3mm_Bridged2Bar_RoundedPad1.0x1.5mm"
-			(at 130.81 107.95 0)
+			(at 130.81 95.25 0)
 			(effects
 				(font
@@
 		)
 		(property "Datasheet" "~"
-			(at 130.81 107.95 0)
+			(at 130.81 95.25 0)
 			(effects
 				(font
@@
 		)
 		(property "Description" "Jumper, 2-pole, closed/bridged"
-			(at 130.81 107.95 0)
+			(at 130.81 95.25 0)
 			(effects
 				(font
@@
 		)
 		(instances
-			(project ""
+			(project "AudioPlayground_HeadsetShield"
 				(path "/f5706b07-e2a9-4776-86c6-e4c8afad03ec"
 					(reference "JP1")

Commit message: Fix Joystick
Connections:
- net BTN4: now also SW6.3; no longer SW6.6
- net BTN5: now also SW6.6; no longer SW6.3
Changed lines of the file:
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@@
 		)
 	)
-	(label "BTN5"
+	(label "BTN4"
 		(at 137.16 135.89 0)
 		(effects
@@
 			)
 			(justify left bottom)
+		)
+	)
+	(label "BTN5"
+		(at 172.72 125.73 180)
+		(effects
+			(font
+				(size 1.27 1.27)
+			)
+			(justify right bottom)
 		)
 	)
@@
 		)
 	)
-	(label "BTN4"
-		(at 172.72 125.73 180)
-		(effects
-			(font
-				(size 1.27 1.27)
-			)
-			(justify right bottom)
-		)
-	)

Commit message: Improve Optic
Other:
- title: (none) -> HeadsetShield
Changed lines of the file:
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@@
 	(generator_version "9.0")
 	(paper "A4")
+	(title_block
+		(title "HeadsetShield")
+		(rev "2.0")
+	)
 	(text "Line In\n"
 		(exclude_from_sim no)
