File: pcbs/AudioPlayground/interface_mcu.kicad_sch (KiCad schematic)
At the start: 21 parts, among them J4 TC2030, U2 R7FA4M2AB3CNE, Y2 12mHz

Commit message: Add LCSC and fix RF
Parts:
- C21, C27, C28, C29, C30: value 100n -> 100nF; LCSC (none) -> C1525
- C22, C24: value 10p -> 10pF; LCSC (none) -> C32949
- C26: LCSC (none) -> C15525
- R18: LCSC (none) -> C25082
- R20, R21, R22, R4, R5: LCSC (none) -> C25744
- R30, R31, R32, R33: value 150 -> 150R; LCSC (none) -> C25082
- U2: LCSC (none) -> R7FA4M2AB3CNE
Changed lines of the file:
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@@
 			)
 		)
-		(property "Value" "100n"
-			(at 153.162 30.48 0)
+		(property "Value" "100nF"
+			(at 152.654 30.48 0)
 			(effects
 				(font
@@
 			)
 		)
+		(property "LCSC" "C1525"
+			(at 152.4 27.94 0)
+			(effects
+				(font
+					(size 1.27 1.27)
+				)
+				(hide yes)
+			)
+		)
 		(pin "2"
 		)
@@
 			)
 		)
-		(property "Value" "100n"
-			(at 146.812 30.48 0)
+		(property "Value" "100nF"
+			(at 146.304 30.48 0)
 			(effects
 				(font
@@
 			)
 		)
+		(property "LCSC" "C1525"
+			(at 146.05 27.94 0)
+			(effects
+				(font
+					(size 1.27 1.27)
+				)
+				(hide yes)
+			)
+		)
 		(pin "2"
 		)
@@
 			)
 		)
+		(property "LCSC" "C25744"
+			(at 124.46 143.51 90)
+			(effects
+				(font
+					(size 1.27 1.27)
+				)
+				(hide yes)
+			)
+		)
 		(pin "2"
 		)
@@
 			)
 		)
-		(property "Value" "10p"
+		(property "Value" "10pF"
 			(at 51.562 94.742 0)
 			(effects
@@
 			)
 		)
+		(property "LCSC" "C32949"
+			(at 50.8 92.71 0)
+			(effects
+				(font
+					(size 1.27 1.27)
+				)
+				(hide yes)
+			)
+		)
 		(pin "2"
 		)
@@
 			)
 		)
-		(property "Value" "150"
-			(at 205.232 62.738 90)
+		(property "Value" "150R"
+			(at 205.994 62.484 90)
 			(effects
 				(font
@@
 			)
 		)
+		(property "LCSC" "C25082"
+			(at 200.66 63.5 90)
+			(effects
+				(font
+					(size 1.27 1.27)
+				)
+				(hide yes)
+			)
+		)
 		(pin "2"
 		)
@@
 			)
 		)
-		(property "Value" "150"
-			(at 205.232 70.358 90)
+		(property "Value" "150R"
+			(at 205.994 70.104 90)
 			(effects
 				(font
@@
 			)
 		)
+		(property "LCSC" "C25082"
+			(at 200.66 71.12 90)
+			(effects
+				(font
+					(size 1.27 1.27)
+				)
+				(hide yes)
+			)
+		)
 		(pin "1"
 		)
@@
 			)
 		)
-		(property "Value" "100n"
-			(at 165.862 30.48 0)
+		(property "Value" "100nF"
+			(at 165.354 30.48 0)
 			(effects
 				(font
@@
 			)
 		)
+		(property "LCSC" "C1525"
+			(at 165.1 27.94 0)
+			(effects
+				(font
+					(size 1.27 1.27)
+				)
+				(hide yes)
+			)
+		)
 		(pin "2"
 		)
@@
 			)
 		)
-		(property "Value" "10p"
+		(property "Value" "10pF"
 			(at 64.008 95.25 0)
 			(effects
@@
 			)
 		)
+		(property "LCSC" "C32949"
+			(at 63.5 92.71 0)
+			(effects
+				(font
+					(size 1.27 1.27)
+				)
+				(hide yes)
+			)
+		)
 		(pin "2"
 		)
@@
 			)
 		)
+		(property "LCSC" "C15525"
+			(at 139.7 27.94 0)
+			(effects
+				(font
+					(size 1.27 1.27)
+				)
+				(hide yes)
+			)
+		)
 		(pin "2"
 		)
@@
 			)
 		)
-		(property "Value" "100n"
-			(at 159.512 30.48 0)
+		(property "Value" "100nF"
+			(at 159.004 30.48 0)
 			(effects
 				(font
@@
 			)
 		)
+		(property "LCSC" "C1525"
+			(at 158.75 27.94 0)
+			(effects
+				(font
+					(size 1.27 1.27)
+				)
+				(hide yes)
+			)
+		)
 		(pin "2"
 		)
@@
 			)
 		)
-		(property "Value" "100n"
+		(property "Value" "100nF"
 			(at 50.8 58.42 90)
 			(effects
@@
 			)
 		)
+		(property "LCSC" "C1525"
+			(at 50.8 63.5 90)
+			(effects
+				(font
+					(size 1.27 1.27)
+				)
+				(hide yes)
+			)
+		)
 		(pin "1"
 		)
@@
 			)
 		)
+		(property "LCSC" "C25744"
+			(at 50.8 71.12 90)
+			(effects
+				(font
+					(size 1.27 1.27)
+				)
+				(hide yes)
+			)
+		)
 		(pin "2"
 		)
@@
 			)
 		)
+		(property "LCSC" "C25744"
+			(at 77.47 91.44 90)
+			(effects
+				(font
+					(size 1.27 1.27)
+				)
+				(hide yes)
+			)
+		)
 		(pin "1"
 		)
@@
 			)
 		)
+		(property "LCSC" "C25082"
+			(at 218.44 101.6 90)
+			(effects
+				(font
+					(size 1.27 1.27)
+				)
+				(hide yes)
+			)
+		)
 		(pin "2"
 		)
@@
 			)
 		)
-		(property "Value" "150"
-			(at 205.232 67.564 90)
+		(property "Value" "150R"
+			(at 205.994 67.31 90)
 			(effects
 				(font
@@
 			)
 		)
+		(property "LCSC" "C25082"
+			(at 200.66 68.58 90)
+			(effects
+				(font
+					(size 1.27 1.27)
+				)
+				(hide yes)
+			)
+		)
 		(pin "1"
 		)
@@
 			)
 		)
+		(property "LCSC" "C25744"
+			(at 130.81 127 0)
+			(effects
+				(font
+					(size 1.27 1.27)
+				)
+				(hide yes)
+			)
+		)
 		(pin "2"
 		)
@@
 			)
 		)
+		(property "LCSC" "C25744"
+			(at 133.35 127 0)
+			(effects
+				(font
+					(size 1.27 1.27)
+				)
+				(hide yes)
+			)
+		)
 		(pin "2"
 		)
@@
 			)
 		)
+		(property "LCSC" "R7FA4M2AB3CNE"
+			(at 91.44 40.64 0)
+			(effects
+				(font
+					(size 1.27 1.27)
+				)
+				(hide yes)
+			)
+		)
 		(pin "1"
 		)
@@
 			)
 		)
-		(property "Value" "150"
-			(at 205.232 65.278 90)
+		(property "Value" "150R"
+			(at 205.994 65.024 90)
 			(effects
 				(font
@@
 			(at 200.66 66.04 90)
 			(effects
+				(font
+					(size 1.27 1.27)
+				)
+				(hide yes)
+			)
+		)
+		(property "LCSC" "C25082"
+			(at 200.66 66.04 90)
+			(effects

Commit message: Fix values
Parts:
- C26: value 10u -> 10uF
Changed lines of the file:
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@@
 			)
 		)
-		(property "Value" "10u"
+		(property "Value" "10uF"
 			(at 140.462 30.48 0)
 			(effects

Commit message: Update MICs
Parts:
- removed R32: 150R, Resistor_SMD:R_0402_1005Metric, symbol Device:R
- U2: LCSC R7FA4M2AB3CNE -> C3226797
- Y2: LCSC (none) -> C2901648
Connections:
- net P100: no longer names the net of U2.36 (P100)
- no-connect marks 16 -> 17
Changed lines of the file:
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@@
 	)
 	(no_connect
+		(at 170.18 63.5)
+	)
+	(no_connect
 		(at 123.19 110.49)
 	)
@@
 	)
 	(bus_entry
-		(at 226.06 71.12)
-		(size -2.54 -2.54)
-		(stroke
-			(width 0)
-			(type default)
-		)
-	)
-	(bus_entry
 		(at 223.52 63.5)
 		(size 2.54 2.54)
@@
 	(wire
 		(pts
-			(xy 204.47 68.58) (xy 223.52 68.58)
-		)
-		(stroke
-			(width 0)
-			(type default)
-		)
-	)
-	(wire
-		(pts
 			(xy 146.05 24.13) (xy 152.4 24.13)
 		)
@@
 	(wire
 		(pts
-			(xy 194.31 68.58) (xy 196.85 68.58)
-		)
-		(stroke
-			(width 0)
-			(type default)
-		)
-	)
-	(bus
-		(pts
-			(xy 226.06 68.58) (xy 226.06 71.12)
-		)
-		(stroke
-			(width 0)
-			(type default)
-		)
-	)
-	(wire
-		(pts
 			(xy 118.11 110.49) (xy 118.11 119.38)
 		)
@@
 	(bus
 		(pts
-			(xy 226.06 71.12) (xy 226.06 73.66)
+			(xy 226.06 68.58) (xy 226.06 73.66)
 		)
 		(stroke
@@
 		)
 	)
-	(label "P100"
-		(at 170.18 63.5 0)
-		(effects
-			(font
-				(size 1.27 1.27)
-			)
-			(justify left bottom)
-		)
-	)
 	(label "SWD.SWDCLK"
 		(at 209.55 66.04 0)
@@
 		)
 	)
-	(label "P100"
-		(at 194.31 68.58 180)
-		(effects
-			(font
-				(size 1.27 1.27)
-			)
-			(justify right bottom)
-		)
-	)
-	(label "SWD.SWO"
-		(at 209.55 68.58 0)
-		(effects
-			(font
-				(size 1.27 1.27)
-			)
-			(justify left bottom)
-		)
-	)
 	(label "P301"
 		(at 222.25 99.06 0)
@@
 			)
 		)
+		(property "LCSC" "C2901648"
+			(at 57.15 87.63 0)
+			(effects
+				(font
+					(size 1.27 1.27)
+				)
+				(hide yes)
+			)
+		)
 		(pin "2"
 		)
@@
 	(symbol
 		(lib_id "Device:R")
-		(at 200.66 68.58 90)
-		(unit 1)
-		(exclude_from_sim no)
-		(in_bom yes)
-		(on_board yes)
-		(dnp no)
-		(property "Reference" "R32"
-			(at 200.914 68.58 90)
-			(effects
-				(font
-					(size 1.27 1.27)
-				)
-			)
-		)
-		(property "Value" "150R"
-			(at 205.994 67.31 90)
-			(effects
-				(font
-					(size 1.27 1.27)
-				)
-			)
-		)
-		(property "Footprint" "Resistor_SMD:R_0402_1005Metric"
-			(at 200.66 70.358 90)
-			(effects
-				(font
-					(size 1.27 1.27)
-				)
-				(hide yes)
-			)
-		)
-		(property "Datasheet" "~"
-			(at 200.66 68.58 0)
-			(effects
-				(font
-					(size 1.27 1.27)
-				)
-				(hide yes)
-			)
-		)
-		(property "Description" "Resistor"
-			(at 200.66 68.58 0)
-			(effects
-				(font
-					(size 1.27 1.27)
-				)
-				(hide yes)
-			)
-		)
-		(property "MOUSER" " 603-RC0402FR-7D150RL "
-			(at 200.66 68.58 90)
-			(effects
-				(font
-					(size 1.27 1.27)
-				)
-				(hide yes)
-			)
-		)
-		(property "LCSC" "C25082"
-			(at 200.66 68.58 90)
-			(effects
-				(font
-					(size 1.27 1.27)
-				)
-				(hide yes)
-			)
-		)
-		(pin "1"
-		)
-		(pin "2"
-		)
-		(instances
-			(project "MasterProject"
-				(path "/1c455b59-0247-4883-9aca-444b4cb10447/fa0718d0-305f-456b-934a-4cd39d3c1c9c"
-					(reference "R32")
-					(unit 1)
-				)
-			)
-		)
-	)
-	(symbol
-		(lib_id "Device:R")
 		(at 130.81 127 0)
 		(unit 1)
@@
 			)
 		)
-		(property "LCSC" "R7FA4M2AB3CNE"
+		(property "LCSC" "C3226797"
 			(at 91.44 40.64 0)
 			(effects

Commit message: Improve Optic
Other:
- title: (none) -> LE Audio Playground
- moved on the sheet: C21, C22, C24, C26, C27, C28, C29, C30, J4, R18, R20, R21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
