File: pcbs/AudioPlayground/mcu.kicad_sch (KiCad schematic)
At the start: 31 parts, among them U1 nRF5340-QKxx, Y1 32MHz, Y4 32.768kHz

Commit message: updated footprints, added i2s testpoints
Parts:
- TP1: value TestPoint -> SDA
- TP2: value TestPoint -> SCL
Changed lines of the file:
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@@
 			)
 		)
-		(property "Value" "TestPoint"
+		(property "Value" "SDA"
 			(at 181.356 144.018 0)
 			(effects
@@
 			)
 		)
-		(property "Value" "TestPoint"
+		(property "Value" "SCL"
 			(at 181.61 155.702 0)
 			(effects

Commit message: Add LCSC and fix RF
Parts:
- C1: LCSC (none) -> C15195
- C10, C4, C7, C8: value 1.0uF -> 1uF; LCSC (none) -> C52923
- C11, C12, C13, C14, C15, C16, C17, C18, C3, C43: LCSC (none) -> C1525
- C19: LCSC (none) -> C52923
- C20: now not fitted
- C23: LCSC (none) -> C397301
- C5, C6: LCSC (none) -> C23733
- C9: LCSC (none) -> C1531
- L1, L2: LCSC (none) -> C48946156
- L3: LCSC (none) -> C86061
- R1: value 2R2 -> 2.2R; LCSC (none) -> C25101
- R26: LCSC (none) -> C25744
- U1: LCSC (none) -> C3015611

Commit message: Update MICs
Parts:
- Y1: LCSC (none) -> C37635386
- Y4: LCSC (none) -> C99010
Connections:
- net P0.11: no longer names the net of U1.AK4 (CSN/TRACEDATA0/P0.11)
- no-connect marks 8 -> 9
Changed lines of the file:
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@@
 	)
 	(no_connect
+		(at 138.43 78.74)
+	)
+	(no_connect
 		(at 138.43 162.56)
 	)
@@
 	)
 	(bus_entry
+		(at 259.08 120.65)
+		(size -2.54 -2.54)
+		(stroke
+			(width 0)
+			(type default)
+		)
+	)
+	(bus_entry
 		(at 256.54 55.88)
 		(size 2.54 2.54)
@@
 	)
 	(bus_entry
-		(at 259.08 125.73)
-		(size -2.54 -2.54)
-		(stroke
-			(width 0)
-			(type default)
-		)
-	)
-	(bus_entry
 		(at 259.08 97.79)
 		(size -2.54 -2.54)
@@
 	)
 	(bus_entry
+		(at 256.54 120.65)
+		(size 2.54 2.54)
+		(stroke
+			(width 0)
+			(type default)
+		)
+	)
+	(bus_entry
 		(at 256.54 48.26)
 		(size 2.54 2.54)
@@
 	)
 	(bus_entry
-		(at 259.08 118.11)
-		(size -2.54 -2.54)
-		(stroke
-			(width 0)
-			(type default)
-		)
-	)
-	(bus_entry
 		(at 191.77 74.93)
 		(size -2.54 -2.54)
@@
 	)
 	(bus_entry
-		(at 256.54 120.65)
-		(size 2.54 2.54)
-		(stroke
-			(width 0)
-			(type default)
-		)
-	)
-	(bus_entry
 		(at 256.54 102.87)
 		(size 2.54 2.54)
@@
 	)
 	(bus_entry
-		(at 256.54 118.11)
-		(size 2.54 2.54)
+		(at 256.54 149.86)
+		(size -2.54 -2.54)
 		(stroke
 			(width 0)
@@
 	)
 	(bus_entry
-		(at 256.54 149.86)
+		(at 259.08 36.83)
 		(size -2.54 -2.54)
 		(stroke
@@
 	)
 	(bus_entry
-		(at 259.08 36.83)
+		(at 191.77 99.06)
 		(size -2.54 -2.54)
 		(stroke
@@
 	)
 	(bus_entry
-		(at 191.77 99.06)
-		(size -2.54 -2.54)
+		(at 256.54 123.19)
+		(size 2.54 2.54)
 		(stroke
 			(width 0)
@@
 		)
 	)
-	(bus
-		(pts
-			(xy 259.08 118.11) (xy 259.08 120.65)
-		)
-		(stroke
-			(width 0)
-			(type default)
-		)
-	)
-	(wire
-		(pts
-			(xy 243.84 120.65) (xy 256.54 120.65)
-		)
-		(stroke
-			(width 0)
-			(type default)
-		)
-	)
 	(polyline
 		(pts
@@
 	(wire
 		(pts
+			(xy 243.84 120.65) (xy 256.54 120.65)
+		)
+		(stroke
+			(width 0)
+			(type default)
+		)
+	)
+	(wire
+		(pts
 			(xy 50.8 111.76) (xy 67.31 111.76)
 		)
@@
 	(bus
 		(pts
-			(xy 259.08 123.19) (xy 259.08 120.65)
+			(xy 259.08 120.65) (xy 259.08 123.19)
 		)
 		(stroke
@@
 		)
 	)
+	(wire
+		(pts
+			(xy 243.84 123.19) (xy 256.54 123.19)
+		)
+		(stroke
+			(width 0)
+			(type default)
+		)
+	)
 	(bus
 		(pts
@@
 		)
 	)
-	(wire
-		(pts
-			(xy 241.3 123.19) (xy 256.54 123.19)
-		)
-		(stroke
-			(width 0)
-			(type default)
-		)
-	)
 	(bus
 		(pts
@@
 		)
 	)
-	(bus
-		(pts
-			(xy 259.08 123.19) (xy 259.08 125.73)
-		)
-		(stroke
-			(width 0)
-			(type default)
-		)
-	)
 	(wire
 		(pts
@@
 		)
 	)
-	(wire
+	(polyline
 		(pts
-			(xy 243.84 115.57) (xy 256.54 115.57)
+			(xy 145.415 163.195) (xy 145.415 172.085)
 		)
 		(stroke
@@
 		)
 	)
-	(polyline
+	(wire
 		(pts
-			(xy 145.415 163.195) (xy 145.415 172.085)
+			(xy 180.34 151.13) (xy 194.31 151.13)
 		)
 		(stroke
@@
 	(wire
 		(pts
-			(xy 180.34 151.13) (xy 194.31 151.13)
+			(xy 241.3 63.5) (xy 256.54 63.5)
 		)
 		(stroke
@@
 	(wire
 		(pts
-			(xy 241.3 63.5) (xy 256.54 63.5)
+			(xy 50.8 110.49) (xy 50.8 111.76)
 		)
 		(stroke
@@
 		)
 	)
-	(wire
+	(bus
 		(pts
-			(xy 50.8 110.49) (xy 50.8 111.76)
+			(xy 259.08 123.19) (xy 259.08 125.73)
 		)
 		(stroke
@@
 		)
 	)
-	(bus
+	(wire
 		(pts
-			(xy 256.54 165.1) (xy 256.54 162.56)
+			(xy 243.84 118.11) (xy 256.54 118.11)
 		)
 		(stroke
@@
 		)
 	)
-	(wire
+	(bus
 		(pts
-			(xy 52.07 55.88) (xy 72.39 55.88)
+			(xy 256.54 165.1) (xy 256.54 162.56)
 		)
 		(stroke
@@
 		)
 	)
-	(polyline
+	(wire
 		(pts
-			(xy 144.78 53.975) (xy 144.78 65.405)
+			(xy 52.07 55.88) (xy 72.39 55.88)
 		)
 		(stroke
@@
 		)
 	)
-	(wire
+	(polyline
 		(pts
-			(xy 123.19 19.05) (xy 130.81 19.05)
+			(xy 144.78 53.975) (xy 144.78 65.405)
 		)
 		(stroke
@@
 	(wire
 		(pts
-			(xy 243.84 118.11) (xy 256.54 118.11)
+			(xy 123.19 19.05) (xy 130.81 19.05)
 		)
 		(stroke
@@
 		)
 	)
-	(label "P0.11"
-		(at 241.3 123.19 180)
-		(effects
-			(font
-				(size 1.27 1.27)
-			)
-			(justify right bottom)
-		)
-	)
 	(label "P0.25"
 		(at 241.3 71.12 180)
@@
 		)
 	)
+	(label "SWD.SWDIO"
+		(at 243.84 120.65 0)
+		(effects
+			(font
+				(size 1.27 1.27)
+			)
+			(justify left bottom)
+		)
+	)
 	(label "A5"
 		(at 246.38 73.66 0)
@@
 		)
 	)
-	(label "SWD.SWDIO"
-		(at 243.84 118.11 0)
-		(effects
-			(font
-				(size 1.27 1.27)
-			)
-			(justify left bottom)
-		)
-	)
 	(label "Codec.SDA"
 		(at 182.88 148.59 0)
@@
 		)
 	)
-	(label "SWD.RESET"
-		(at 243.84 115.57 0)
-		(effects
-			(font
-				(size 1.27 1.27)
-			)
-			(justify left bottom)
-		)
-	)
 	(label "P0.04"
 		(at 241.3 60.96 180)
@@
 		)
 	)
-	(label "SWD.SWDCLK"
-		(at 243.84 120.65 0)
+	(label "SWD.RESET"
+		(at 243.84 118.11 0)
 		(effects
 			(font
@@
 		)
 	)
+	(label "SWD.SWDCLK"
+		(at 243.84 123.19 0)
+		(effects
+			(font
+				(size 1.27 1.27)
+			)
+			(justify left bottom)
+		)
+	)
 	(label "P0.08"
 		(at 241.3 34.29 180)
@@
 		)
 	)
-	(label "SWD.SWO"
-		(at 243.84 123.19 0)
-		(effects
-			(font
-				(size 1.27 1.27)
-			)
-			(justify left bottom)
-		)
-	)
 	(label "P0.30"
 		(at 138.43 127 0)
@@
 		)
 	)
-	(label "P0.11"
-		(at 138.43 78.74 0)
-		(effects
-			(font
-				(size 1.27 1.27)
-			)
-			(justify left bottom)
-		)
-	)
 	(label "P0.19"
 		(at 242.57 160.02 180)
@@
 			)
 		)
+		(property "LCSC" "C99010"
+			(at 166.37 52.07 90)
+			(effects
+				(font
+					(size 1.27 1.27)
+				)
+				(hide yes)
+			)
+		)
 		(pin "1"
 		)
@@
 			(at 63.5 78.74 90)
 			(effects
+				(font
+					(size 1.27 1.27)
+				)
+				(hide yes)
+			)
+		)
+		(property "LCSC" "C37635386"
+			(at 63.5 78.74 90)
+			(effects

Commit message: Fix Codec IRQ
Connections:
- net CODECIRQ: now reaches U1.AK4 (CSN/TRACEDATA0/P0.11)
- no-connect marks 9 -> 8
Other:
- note removed: "SWD"
Changed lines of the file:
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@@
 		)
 	)
-	(text "SWD\n"
-		(exclude_from_sim no)
-		(at 146.304 77.47 90)
-		(effects
-			(font
-				(size 1.27 1.27)
-			)
-		)
-	)
 	(text "RGB1"
 		(exclude_from_sim no)
@@
 	)
 	(no_connect
-		(at 138.43 78.74)
-	)
-	(no_connect
 		(at 138.43 162.56)
 	)
@@
 	(wire
 		(pts
+			(xy 138.43 78.74) (xy 146.05 78.74)
+		)
+		(stroke
+			(width 0)
+			(type default)
+		)
+	)
+	(wire
+		(pts
 			(xy 176.53 96.52) (xy 189.23 96.52)
 		)
@@
 		)
 	)
-	(polyline
-		(pts
-			(xy 144.78 76.835) (xy 144.78 78.74)
-		)
-		(stroke
-			(width 0)
-			(type default)
-		)
-	)
 	(wire
 		(pts
@@
 		(effects
 			(font
+				(size 1.27 1.27)
+			)
+			(justify left)
+		)
+	)
+	(hierarchical_label "CODECIRQ"
+		(shape input)
+		(at 146.05 78.74 0)
+		(effects
+			(font

Commit message: V2.1
Parts:
- added TP8: SWDIO, TestPoint:TestPoint_Pad_D1.0mm, symbol Connector:TestPoint
- added TP9: SWDCLK, TestPoint:TestPoint_Pad_D1.0mm, symbol Connector:TestPoint
Connections:
- net SWD.SWDCLK: now also TP9.1
- net SWD.SWDIO: now also TP8.1
Changed lines of the file:
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@@
 		)
 	)
+	(wire
+		(pts
+			(xy 232.41 123.19) (xy 256.54 123.19)
+		)
+		(stroke
+			(width 0)
+			(type default)
+		)
+	)
 	(polyline
 		(pts
@@
 	(wire
 		(pts
-			(xy 243.84 120.65) (xy 256.54 120.65)
-		)
-		(stroke
-			(width 0)
-			(type default)
-		)
-	)
-	(wire
-		(pts
 			(xy 50.8 111.76) (xy 67.31 111.76)
 		)
@@
 		)
 	)
-	(wire
-		(pts
-			(xy 243.84 123.19) (xy 256.54 123.19)
-		)
-		(stroke
-			(width 0)
-			(type default)
-		)
-	)
 	(bus
 		(pts
@@
 	(wire
 		(pts
+			(xy 238.76 120.65) (xy 256.54 120.65)
+		)
+		(stroke
+			(width 0)
+			(type default)
+		)
+	)
+	(wire
+		(pts
 			(xy 67.31 111.76) (xy 72.39 111.76)
 		)
@@
 	)
 	(symbol
+		(lib_id "Connector:TestPoint")
+		(at 238.76 120.65 90)
+		(unit 1)
+		(exclude_from_sim no)
+		(in_bom no)
+		(on_board yes)
+		(dnp no)
+		(fields_autoplaced yes)
+		(property "Reference" "TP8"
+			(at 235.458 115.57 90)
+			(effects
+				(font
+					(size 1.27 1.27)
+				)
+			)
+		)
+		(property "Value" "SWDIO"
+			(at 235.458 118.11 90)
+			(effects
+				(font
+					(size 1.27 1.27)
+				)
+			)
+		)
+		(property "Footprint" "TestPoint:TestPoint_Pad_D1.0mm"
+			(at 238.76 115.57 0)
+			(effects
+				(font
+					(size 1.27 1.27)
+				)
+				(hide yes)
+			)
+		)
+		(property "Datasheet" "~"
+			(at 238.76 115.57 0)
+			(effects
+				(font
+					(size 1.27 1.27)
+				)
+				(hide yes)
+			)
+		)
+		(property "Description" "test point"
+			(at 238.76 120.65 0)
+			(effects
+				(font
+					(size 1.27 1.27)
+				)
+				(hide yes)
+			)
+		)
+		(pin "1"
+		)
+		(instances
+			(project "AudioPlayground"
+				(path "/1c455b59-0247-4883-9aca-444b4cb10447/26d34958-e592-44d3-88a3-daa1680508c2"
+					(reference "TP8")
+					(unit 1)
+				)
+			)
+		)
+	)
+	(symbol
 		(lib_id "power:GND")
 		(at 105.41 190.5 0)
@@
 					(unit 1)
 				)
+			)
+		)
+	)
+	(symbol
+		(lib_id "Connector:TestPoint")
+		(at 232.41 123.19 90)
+		(unit 1)
+		(exclude_from_sim no)
+		(in_bom no)
+		(on_board yes)
+		(dnp no)
+		(fields_autoplaced yes)
+		(property "Reference" "TP9"
+			(at 229.108 118.11 90)
+			(effects
+				(font
+					(size 1.27 1.27)
+				)
+			)
+		)
+		(property "Value" "SWDCLK"
+			(at 229.108 120.65 90)
+			(effects
+				(font
+					(size 1.27 1.27)
+				)
+			)
+		)
+		(property "Footprint" "TestPoint:TestPoint_Pad_D1.0mm"
+			(at 232.41 118.11 0)
+			(effects
+				(font
+					(size 1.27 1.27)
+				)
+				(hide yes)
+			)
+		)
+		(property "Datasheet" "~"
+			(at 232.41 118.11 0)
+			(effects
+				(font
+					(size 1.27 1.27)
+				)
+				(hide yes)
+			)
+		)
+		(property "Description" "test point"
+			(at 232.41 123.19 0)
+			(effects
+				(font
+					(size 1.27 1.27)
+				)
+				(hide yes)
+			)
+		)
+		(pin "1"
+		)
+		(instances
+			(project "AudioPlayground"
+				(path "/1c455b59-0247-4883-9aca-444b4cb10447/26d34958-e592-44d3-88a3-daa1680508c2"
+					(reference "TP9")
+					(unit 1)
+				)

Commit message: Improve Optic
Other:
- note added: "LED0"
- note added: "LED1"
- note added: "LED2"
- note removed: "LED"
- note removed: "Note: FLIPPED SDIN and SDOUT"
- note removed: "Note: FLIPPED i2c pins"
- note removed: "Note: Fixed SWDIO/SWDCLK"
- title: (none) -> LE Audio Playground
- moved on the sheet: C1, C10, C11, C12, C13, C14, C15, C16, C17, C18, C19, C20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
